Commit message: Second commit

File: src/mybot_description/urdf/mybot.xacro (robot description, xacro)
@@ -124,6 +124,6 @@
     <parent link="chassis"/>
     <axis xyz="0 1 0" rpy="0 0 0"/>
-    <limit effort="100" velocity="100"/>
-    <joint_properties damping="0.0" friction="1.0"/>
+    <!--limit effort="100" velocity="100"/>
+    <joint_properties damping="0.0" friction="1.0"/-->
   </joint>
   <joint type="continuous" name="right_wheel_hinge">
@@ -132,6 +132,6 @@
     <parent link="chassis"/>
     <axis xyz="0 1 0" rpy="0 0 0"/>
-    <limit effort="100" velocity="100"/>
-    <joint_properties damping="0.0" friction="1.0"/>
+    <!--limit effort="100" velocity="100"/>
+    <joint_properties damping="0.0" friction="1.0"/-->
   </joint>
  <joint type="continuous" name="left_wheel_back_hinge">
@@ -140,6 +140,6 @@
     <parent link="chassis"/>
     <axis xyz="0 1 0" rpy="0 0 0"/>
-    <limit effort="100" velocity="100"/>
-    <joint_properties damping="0.0" friction="1.0"/>
+    <!--limit effort="100" velocity="100"/>
+    <joint_properties damping="0.0" friction="1.0"/-->
   </joint>
   <joint type="continuous" name="right_wheel_back_hinge">
@@ -148,6 +148,6 @@
     <parent link="chassis"/>
     <axis xyz="0 1 0" rpy="0 0 0"/>
-    <limit effort="100" velocity="100"/>
-    <joint_properties damping="0.0" friction="1.0"/>
+    <!--limit effort="100" velocity="100"/>
+    <joint_properties damping="0.0" friction="1.0"/-->
   </joint>
 </robot>
